File: hardware/pihat_template.sch (KiCad schematic (older format))
At the start: 29 parts, among them P1 CONN_01X02, P2 CONN_01X02, P3 Raspberry_Pi_+_Conn, U1 LM3489, U2 CAT24C32HU4I-GT3, U3 FDC5614P, U4 LM1117IMPX-ADJ

Commit message: add ground
Connections:
- wire segments 99 -> 143
