File: hardware/Ideal_Diode.sch (KiCad schematic (older format))
At the start: 4 parts, among them Q1 BSS138, U5 DMMT5401

Commit message: change some resistors and capacitors form factor to 0805
Parts:
- R11, R12: footprint project:r_0402 -> Resistors_SMD:R_0805
Changed lines of the file:
@@
 F 0 "R12" V 6280 4800 50  0000 C CNN
 F 1 "47k" V 6207 4801 50  0000 C CNN
-F 2 "project:r_0402" V 6130 4800 30  0001 C CNN
+F 2 "Resistors_SMD:R_0805" V 6130 4800 30  0001 C CNN
 F 3 "" H 6200 4800 30  0000 C CNN
 F 4 "667-ERJ-2RKF4702X" V 6200 4800 60  0001 C CNN "Mouser Part No."
@@
 F 0 "R11" V 5880 4800 50  0000 C CNN
 F 1 "10k" V 5807 4801 50  0000 C CNN
-F 2 "project:r_0402" V 5730 4800 30  0001 C CNN
+F 2 "Resistors_SMD:R_0805" V 5730 4800 30  0001 C CNN
 F 3 "" H 5800 4800 30  0000 C CNN
 F 4 "71-CRCW0402-10K-E3" V 5800 4800 60  0001 C CNN "Mouser Part No."

Commit message: replaced r and c footprints with project:r_805 and project:c_805
Parts:
- R11, R12: footprint Resistors_SMD:R_0805 -> project:r_0805
Changed lines of the file:
@@
 F 0 "R12" V 6280 4800 50  0000 C CNN
 F 1 "47k" V 6207 4801 50  0000 C CNN
-F 2 "Resistors_SMD:R_0805" V 6130 4800 30  0001 C CNN
+F 2 "project:r_0805" V 6130 4800 30  0001 C CNN
 F 3 "" H 6200 4800 30  0000 C CNN
 F 4 "667-ERJ-2RKF4702X" V 6200 4800 60  0001 C CNN "Mouser Part No."
@@
 F 0 "R11" V 5880 4800 50  0000 C CNN
 F 1 "10k" V 5807 4801 50  0000 C CNN
-F 2 "Resistors_SMD:R_0805" V 5730 4800 30  0001 C CNN
+F 2 "project:r_0805" V 5730 4800 30  0001 C CNN
 F 3 "" H 5800 4800 30  0000 C CNN
 F 4 "71-CRCW0402-10K-E3" V 5800 4800 60  0001 C CNN "Mouser Part No."

Commit message: created DMMT5401 footprint and updated netlist
Parts:
- U5: footprint project:sot23-6 -> project:DMMT5401-7F
Changed lines of the file:
@@
 F 0 "U5" H 5700 4150 47  0000 C CNN
 F 1 "DMMT5401" H 6450 3800 47  0000 C CNN
-F 2 "project:sot23-6" H 5850 3700 47  0001 C CNN
+F 2 "project:DMMT5401-7F" H 5850 3700 47  0001 C CNN
 F 3 "" H 5850 3700 47  0000 C CNN
 F 4 "621-DMMT5401-7-F" H 6000 4000 60  0001 C CNN "Mouser Part No."

Commit message: partial update of components refs. for buiding a better BOM
Parts:
- Q1: Farnell Part No. 9845330 -> (none); Part Number (none) -> 9845330; Supplier (none) -> Farnell
- R11: Farnell Part No. 2324717 -> (none); Part Number (none) -> 2447553; Supplier (none) -> Farnell
- R12: Farnell Part No. 6379860 -> (none); Part Number (none) -> 2447664; Supplier (none) -> Farnell
- U5: Farnell Part No. 1773583 -> (none); Part Number (none) -> 1773583; Supplier (none) -> Farnell
Changed lines of the file:
@@
 F 3 "" H 6000 3100 60  0000 C CNN
 F 4 "621-DMG2305UX-13" H 6000 3100 60  0001 C CNN "Mouser Part No."
-F 5 "9845330" H 6000 3100 60  0001 C CNN "Farnell Part No."
+F 5 "Farnell" H 6000 3100 60  0001 C CNN "Supplier"
+F 6 "9845330" H 6000 3100 60  0001 C CNN "Part Number"
 	1    6000 3100
 	0    -1   -1   0
@@
 F 3 "" H 5850 3700 47  0000 C CNN
 F 4 "621-DMMT5401-7-F" H 6000 4000 60  0001 C CNN "Mouser Part No."
-F 5 "1773583" H 6000 4000 60  0001 C CNN "Farnell Part No."
+F 5 "Farnell" H 6000 4000 60  0001 C CNN "Supplier"
+F 6 "1773583" H 6000 4000 60  0001 C CNN "Part Number"
 	1    6000 4000
 	1    0    0    -1
@@
 F 3 "" H 6200 4800 30  0000 C CNN
 F 4 "667-ERJ-2RKF4702X" V 6200 4800 60  0001 C CNN "Mouser Part No."
-F 5 "6379860" V 6200 4800 60  0001 C CNN "Farnell Part No."
+F 5 "Farnell" V 6200 4800 60  0001 C CNN "Supplier"
+F 6 "2447664" V 6200 4800 60  0001 C CNN "Part Number"
 	1    6200 4800
 	1    0    0    -1
@@
 F 3 "" H 5800 4800 30  0000 C CNN
 F 4 "71-CRCW0402-10K-E3" V 5800 4800 60  0001 C CNN "Mouser Part No."
-F 5 "2324717" V 5800 4800 60  0001 C CNN "Farnell Part No."
+F 5 "Farnell" V 5800 4800 60  0001 C CNN "Supplier"
+F 6 "2447553" V 5800 4800 60  0001 C CNN "Part Number"
 	1    5800 4800
 	1    0    0    -1
